Commit message: Have initial creation of xacro file for arm.

File: homework2/config/twoarm.urdf.xacro (robot description, xacro)
@@ -20,5 +20,5 @@
 <joint name="joint1" type="continuous">
     <axis xyz="0 0 1" />
-    <origin xyz="0 0 0" rpy="0 0 0" />
+    <origin xyz="0 0 0.05" rpy="0 0 0" />
     <parent link="base_link" />
     <child link="arm1" />
@@ -26,7 +26,7 @@
 <link name="arm1">
     <visual>
-    <origin xyz="1 0 0" rpy="0.8 1.6 0.8" />
+    <origin xyz="0.75 0 0" rpy="0.8 1.6 0.8" />
         <geometry>
-            <cylinder radius="0.2" length="2.0"/>
+            <cylinder radius="0.1" length="1.5"/>
         </geometry>
         <material name="green_mat">
@@ -37,5 +37,5 @@
 <joint name ="joint2" type="continuous">
     <axis xyz="0 0 1" />
-    <origin xyz="2.0 0 0" rpy="0 0 0" />
+    <origin xyz="1.5 0 0" rpy="0 0 0" />
     <parent link="arm1" />
     <child link="arm2" />
@@ -43,7 +43,7 @@
 <link name="arm2">
     <visual>
-    <origin xyz="2 0 0" rpy="0 1.6 0" />
+    <origin xyz="0.5 0 0" rpy="0 1.6 0" />
         <geometry>
-            <cylinder radius="0.2" length="4"/>
+            <cylinder radius="0.1" length="1.0"/>
         </geometry>
         <material name="blue_mat">

Commit message: Creation of arm trajectory node

File: homework2/config/twoarm.urdf.xacro (robot description, xacro)
@@ -22,7 +22,7 @@
     <origin xyz="0 0 0.05" rpy="0 0 0" />
     <parent link="base_link" />
-    <child link="arm1" />
+    <child link="link1" />
 </joint>
-<link name="arm1">
+<link name="link1">
     <visual>
     <origin xyz="0.75 0 0" rpy="0.8 1.6 0.8" />
@@ -38,8 +38,8 @@
     <axis xyz="0 0 1" />
     <origin xyz="1.5 0 0" rpy="0 0 0" />
-    <parent link="arm1" />
-    <child link="arm2" />
+    <parent link="link1" />
+    <child link="link2" />
 </joint>
-<link name="arm2">
+<link name="link2">
     <visual>
     <origin xyz="0.5 0 0" rpy="0 1.6 0" />
@@ -52,3 +52,20 @@
     </visual>
 </link>
+<joint name ="joint3" type="fixed">
+    <axis xyz="0 0 1" />
+    <origin xyz="1.0 0 0" rpy="0 0 0" />
+    <parent link="link2" />
+    <child link="link3" />
+</joint>
+<link name="link3">
+    <visual>
+    <origin xyz="0.5 0 0" rpy="0 1.6 0" />
+        <geometry>
+            <cylinder radius="0.1" length="0.1"/>
+        </geometry>
+        <material name="transparent_mat">
+            <color rgba="1 1 1 0" />
+        </material>
+    </visual>
+</link>
 </robot>

Commit message: Completed arm marker node with markers being drawn and fixed parameters issue in twoarm urdf

File: homework2/config/twoarm.urdf.xacro (robot description, xacro)
@@ -1,6 +1,6 @@
 <?xml version="1.0"?>
 <robot xmlns:xacro="http://wiki.ros.org/wiki/xacro" name="twoarm">
-<xacro:property name="arm" value="$(find homework2/config/arms.yaml" />
-<xacro:property name="dictionary" value="${load_yaml (arm)}" />
+<xacro:property name="arm" value="$(find homework2)/config/arm.yaml" />
+<xacro:property name="dictionary" value="${load_yaml(arm)}" />
 <xacro:property name="L1" value="${dictionary['L1']}" />
 <xacro:property name="L2" value="${dictionary['L2']}" />
@@ -26,7 +26,7 @@
 <link name="link1">
     <visual>
-    <origin xyz="0.75 0 0" rpy="0.8 1.6 0.8" />
+    <origin xyz="${L1/2} 0 0" rpy="${pi/4} ${pi/2} ${pi/4}" />
         <geometry>
-            <cylinder radius="0.1" length="1.5"/>
+            <cylinder radius="${R1}" length="${L1}"/>
         </geometry>
         <material name="green_mat">
@@ -37,5 +37,5 @@
 <joint name ="joint2" type="continuous">
     <axis xyz="0 0 1" />
-    <origin xyz="1.5 0 0" rpy="0 0 0" />
+    <origin xyz="${L1} 0 0" rpy="0 0 0" />
     <parent link="link1" />
     <child link="link2" />
@@ -43,7 +43,7 @@
 <link name="link2">
     <visual>
-    <origin xyz="0.5 0 0" rpy="0 1.6 0" />
+    <origin xyz="${L2/2} 0 0" rpy="0 ${pi/2} 0" />
         <geometry>
-            <cylinder radius="0.1" length="1.0"/>
+            <cylinder radius="${R2}" length="${L2}"/>
         </geometry>
         <material name="blue_mat">
@@ -54,5 +54,5 @@
 <joint name ="joint3" type="fixed">
     <axis xyz="0 0 1" />
-    <origin xyz="1.0 0 0" rpy="0 0 0" />
+    <origin xyz="${L2} 0 0" rpy="0 0 0" />
     <parent link="link2" />
     <child link="link3" />
@@ -60,7 +60,7 @@
 <link name="link3">
     <visual>
-    <origin xyz="0.5 0 0" rpy="0 1.6 0" />
+    <origin xyz="${L2/2} 0 0" rpy="0 ${pi/2} 0" />
         <geometry>
-            <cylinder radius="0.1" length="0.1"/>
+            <cylinder radius="${R2}" length="0.1"/>
         </geometry>
         <material name="transparent_mat">

Commit message: Added intertia values to robot arm.

File: homework2/config/twoarm.urdf.xacro (robot description, xacro)
@@ -7,4 +7,5 @@
 <xacro:property name="R1" value="${dictionary['R1']}" />
 <xacro:property name="R2" value="${dictionary['R2']}" />
+<xacro:property name="m" value="1" />
 <link name="base_link" >
     <visual>
@@ -33,4 +34,8 @@
             <color rgba="0 1 0 1" />
         </material>
+        <inertial>
+           <mass value="${m}"/>
+           <inertia ixx="1/12*${m}*(3*${R1}**2 + ${L1}**2)" ixy="0.0" ixz="0.0" iyy="1/12*${m}*(3*${R1}**2 + ${L1}**2)" iyz="0.0" izz="1/2*${m}*${R1}**2"/>
+         </inertial>
     </visual>
 </link>
@@ -50,4 +55,8 @@
             <color rgba="0 0 1 1" />
         </material>
+        <inertial>
+           <mass value="${m}"/>
+           <inertia ixx="1/12*${m}*(3*${R2}**2 + ${L2}**2)" ixy="0.0" ixz="0.0" iyy="1/12*${m}*(3*${R2}**2 + ${L2}**2)" iyz="0.0" izz="1/2*${m}*${R2}**2"/>
+         </inertial>
     </visual>
 </link>

Commit message: Added collisions data in urdf

File: homework2/config/twoarm.urdf.xacro (robot description, xacro)
@@ -39,4 +39,9 @@
          </inertial>
     </visual>
+    <collision>
+           <geometry>
+             <cylinder length="${L1}" radius="${R1}"/>
+           </geometry>
+    </collision>
 </link>
 <joint name ="joint2" type="continuous">
@@ -60,4 +65,9 @@
          </inertial>
     </visual>
+    <collision>
+           <geometry>
+             <cylinder length="${L2}" radius="${R2}"/>
+           </geometry>
+    </collision>
 </link>
 <joint name ="joint3" type="fixed">
